File: hw/yabc/yabc.brd (EAGLE design)
At the start: 100 x 100 mm, 60 parts, among them IC1 ATMEGA644A, IC2 LM1117-5V, IC3 FT232RL, J1 DCJ0202, M3/0 BC847ASMD, M4/1 BC847ASMD, M5/2 BC847ASMD, X1 PN61729-S

Commit message: clock worky, der jenks wird sich freuen
Parts:
- removed LED1, LED2, LED3, LED4, LED5, LED6: (no value), led:LED10MM
- added JP1, JP2: (no value), jumper:JP1
- added JP3: (no value), jumper:JP4
- added LED_H3/0, LED_H4/1, LED_H5/2, LED_M3/0, LED_M4/1, LED_M5/2: (no value), led:LED10MM
- moved R12 174.6 mm to (85.0, 28.2), flipped to the bottom, turned to 90 degrees
- moved R14 173.1 mm to (85.2, 71.1), flipped to the bottom, turned to 270 degrees
- moved R13 151.9 mm to (81.1, 32.0), flipped to the bottom, turned to 270 degrees
- moved H3/0 149.6 mm to (82.0, 28.2), flipped to the bottom, turned to 180 degrees
- moved R15 149.2 mm to (82.9, 67.6), flipped to the bottom, turned to 90 degrees
- moved JMP6 143.4 mm to (81.2, 66.8), flipped to the bottom, turned to 180 degrees
- moved JMP5 135.0 mm to (79.4, 32.8), flipped to the bottom, turned to 180 degrees
- moved H4/1 129.9 mm to (48.5, 28.2), flipped to the bottom, turned to 180 degrees
- moved R6 127.7 mm to (54.1, 28.8), flipped to the bottom, turned to 90 degrees
- moved R10 127.3 mm to (52.0, 71.2), flipped to the bottom, turned to 270 degrees
- moved C5 125.0 mm to (63.3, 25.3), flipped to the bottom
- moved H5/2 110.7 mm to (15.4, 28.6), flipped to the bottom, turned to 180 degrees
- moved R11 106.5 mm to (49.7, 67.6), flipped to the bottom, turned to 90 degrees
- moved M3/0 105.4 mm to (81.9, 71.5), flipped to the bottom
- moved R7 102.7 mm to (47.5, 31.9), flipped to the bottom, turned to 270 degrees
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Connections:
- net +5V: now also JP1.2, JP2.2, JP3.1
- net GND: now also JP1.1, JP2.1, JP3.2
- net N$18: now also LED_H4/1.A; no longer LED2.A
- net N$19: now also LED_H4/1.K; no longer LED2.K
- net N$22: now also LED_M5/2.A; no longer LED3.A
- net N$23: now also LED_M5/2.K; no longer LED3.K
- net N$26: now also LED_M4/1.A; no longer LED4.A
- net N$27: now also LED_M4/1.K; no longer LED4.K
- net N$30: now also LED_H3/0.A; no longer LED5.A
- net N$31: now also LED_H3/0.K; no longer LED5.K
- net N$34: now also LED_M3/0.A; no longer LED6.A
- net N$35: now also LED_M3/0.K; no longer LED6.K
- net N$6: now also LED_H5/2.A; no longer LED1.A
- net N$9: now also LED_H5/2.K; no longer LED1.K
- net SCL: now also JP3.4
- net SDA: now also JP3.3
Routing:
- net +5V: track 0.00 -> 427.5 mm, vias 0 -> 6
- net MINUTE5: track 0.00 -> 199.4 mm, vias 0 -> 3
- net MINUTE3: track 0.00 -> 196.7 mm, vias 0 -> 3
- net MINUTE2: track 0.00 -> 192.9 mm, vias 0 -> 3
- net MINUTE4: track 0.00 -> 189.5 mm, vias 0 -> 3
- net MINUTE7: track 0.00 -> 169.3 mm, vias 0 -> 2
- net MINUTE6: track 0.00 -> 169.1 mm, vias 0 -> 2
- net HOUR0: track 0.00 -> 162.6 mm, vias 0 -> 3
- net MINUTE0: track 0.00 -> 158.5 mm, vias 0 -> 3
- net MINUTE1: track 0.00 -> 153.1 mm, vias 0 -> 3
- net HOUR2: track 0.00 -> 145.5 mm, vias 0 -> 3
- net HOUR3: track 0.00 -> 135.7 mm, vias 0 -> 3
- net HOUR5: track 0.00 -> 132.9 mm, vias 0 -> 3
- net HOUR4: track 0.00 -> 131.8 mm, vias 0 -> 3
- net HOUR1: track 0.00 -> 130.9 mm, vias 0 -> 2
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- added copper zone on layer 1, net GND
- added copper zone on layer 16, net GND
Other:
- board text added: "Armin Schlegel, 09.09.14"
- board text added: "Binary Clock V1"
- board text added: "bot"
- board text added: "top"
