File: hw/yabc/yabc.sch (EAGLE design)
At the start: 60 parts, among them IC1 ATMEGA644A, IC2 LM1117-5V, IC3 FT232RL, J1 DCJ0202, M3/0 BC847ASMD, M4/1 BC847ASMD, M5/2 BC847ASMD, X1 PN61729-S

Commit message: clock worky, der jenks wird sich freuen
Parts:
- added JP1, JP2: (no value), jumper:JP1E
- added JP3: (no value), jumper:JP4E
- renumbered LED1 to LED_H5/2, LED2 to LED_H4/1, LED3 to LED_M5/2, LED4 to LED_M4/1, LED5 to LED_H3/0, LED6 to LED_M3/0
Connections:
- net +5V: now also JP1.2, JP2.2, JP3.1
- net GND: now also JP1.1, JP2.1, JP3.2
- net SCL: now also JP3.4
- net SDA: now also JP3.3
